File: eagle/ignition3.brd (EAGLE design)
At the start: 152.4 x 152.4 mm, 26 parts, among them IC1 LM358N, IC2 NE555, J1 PIN2F061.100, J2 PIN2F061.100, J3 PIN2F061.100, J4 PIN2F061.100, Q1 MJ2955, T1 2N3055

Commit message: BOARDS
Parts:
- removed R7, R9: 10k, resistor:0207/10
- removed R8: 30k, resistor:0207/10
- C1: device rcl:C075-042X103 -> rcl:C050-035X075
- R1, R2: device resistor:0207/15 -> resistor:0207/10
- R3, R4: device pot:RJ9W -> pot:B64Y
- R5: device pot:RJ9W -> resistor:0207/10
- R6: value 10k -> 20k; device resistor:0207/12 -> resistor:0207/10
- moved C3 119.2 mm to (57.1, 24.4), turned to 0 degrees
- moved R5 44.9 mm to (41.1, 46.7), turned to 0 degrees
- moved IC1 26.5 mm to (33.8, 129.0)
- moved J1 21.8 mm to (99.1, 22.9)
- moved R6 19.0 mm to (34.8, 104.9), turned to 315 degrees
- moved R1 17.8 mm to (17.0, 106.7), turned to 0 degrees
- moved R2 15.4 mm to (39.9, 110.0), turned to 135 degrees
- moved Q1 14.0 mm to (28.4, 71.6), turned to 90 degrees
- moved J4 12.5 mm to (8.13, 28.2), turned to 270 degrees
- moved C1 10.9 mm to (19.3, 134.9), turned to 0 degrees
- moved C2 10.9 mm to (19.8, 119.6), turned to 270 degrees
- moved C4 10.4 mm to (57.4, 14.7)
- moved R3 6.36 mm to (14.0, 143.5)
- moved T1 5.92 mm to (28.4, 22.9), turned to 90 degrees
- moved C5 4.58 mm to (56.6, 122.4)
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Connections:
- removed net N$10: IC1.5, R6.1, R7.1
- removed net N$11: IC1.6, R8.1, R9.2
- removed net N$4: IC1.7, R1.1, R9.1
- net GND: no longer R7.2
- net N$1: now also R5.2; no longer R5.E
- net N$12: now also R1.1; no longer R8.2
- net N$3: now also R5.1; no longer R5.A, R5.S
- net N$9: now also R6.1
Routing:
- net N$1: track 34.3 -> 100.6 mm
- net -12V: track 144.0 -> 88.6 mm, vias 2 -> 0
- net N$10: track 49.4 -> 0.00 mm
- net N$11: track 24.4 -> 0.00 mm
- net +12V: track 325.7 -> 302.6 mm
- net N$4: track 22.0 -> 0.00 mm
- net N: track 140.4 -> 118.5 mm
- net N$7: track 44.4 -> 34.0 mm
- net N$3: track 88.1 -> 98.2 mm
- net N$6: track 104.7 -> 114.6 mm, vias 2 -> 0
- net N$9: track 11.7 -> 19.4 mm
- net N$12: track 20.4 -> 13.7 mm
- net N$8: track 29.1 -> 24.7 mm
- net N$2: track 12.2 -> 8.69 mm
- added copper zone on layer 1, net GND
