File: eagle/ignition3.sch (EAGLE design)
At the start: 26 parts, among them IC1 LM358N, IC2 NE555, J1 PIN2F061.100, J2 PIN2F061.100, J3 PIN2F061.100, J4 PIN2F061.100, Q1 MJ2955, T1 2N3055

Commit message: BOARDS
Parts:
- removed R7, R9: 10k, resistor:R-US_0207/10
- removed R8: 30k, resistor:R-US_0207/10
- R5: device pot:TRIM_US-B64Y -> resistor:R-US_0207/10
- R6: value 10k -> 20k
Connections:
- removed net N$10: IC1B.+IN, R6.1, R7.1
- removed net N$11: IC1B.-IN, R8.1, R9.2
- removed net N$4: IC1B.OUT, R1.1, R9.1
- net GND: no longer R7.2
- net N$1: now also R5.2; no longer R5.E
- net N$12: now also R1.1; no longer R8.2
- net N$3: now also R5.1; no longer R5.A, R5.S
- net N$9: now also R6.1
Other:
- moved on the sheet: R6
Changed lines of the file:
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@@
 <part name="C6" library="rcl" deviceset="CPOL-US" device="E5-5"/>
 <part name="R2" library="resistor" deviceset="R-US_" device="0207/10" value="10k"/>
-<part name="R5" library="pot" deviceset="TRIM_US-" device="B64Y" value="20k"/>
 <part name="SUPPLY3" library="supply2" deviceset="GND" device=""/>
-<part name="R6" library="resistor" deviceset="R-US_" device="0207/10" value="10k"/>
-<part name="R7" library="resistor" deviceset="R-US_" device="0207/10" value="10k"/>
-<part name="R8" library="resistor" deviceset="R-US_" device="0207/10" value="30k"/>
-<part name="R9" library="resistor" deviceset="R-US_" device="0207/10" value="10k"/>
+<part name="R6" library="resistor" deviceset="R-US_" device="0207/10" value="20k"/>
 <part name="P+7" library="supply1" deviceset="+12V" device=""/>
-<part name="SUPPLY8" library="supply2" deviceset="GND" device=""/>
+<part name="R5" library="resistor" deviceset="R-US_" device="0207/10" value="20k"/>
 </parts>
 <sheets>
@@
 <instance part="C6" gate="G$1" x="-5.08" y="127"/>
 <instance part="R2" gate="G$1" x="5.08" y="48.26"/>
-<instance part="R5" gate="G$1" x="33.02" y="22.86" rot="R90"/>
-<instance part="IC1" gate="B" x="-20.32" y="43.18"/>
 <instance part="SUPPLY3" gate="GND" x="-5.08" y="48.26" rot="R270"/>
-<instance part="R6" gate="G$1" x="-27.94" y="60.96" rot="R90"/>
-<instance part="R7" gate="G$1" x="-33.02" y="45.72" rot="R180"/>
-<instance part="R8" gate="G$1" x="-33.02" y="30.48" rot="R180"/>
-<instance part="R9" gate="G$1" x="-20.32" y="30.48" rot="R180"/>
-<instance part="P+7" gate="1" x="-27.94" y="76.2"/>
-<instance part="SUPPLY8" gate="GND" x="-43.18" y="45.72" rot="R270"/>
+<instance part="R6" gate="G$1" x="12.7" y="53.34" rot="R90"/>
+<instance part="P+7" gate="1" x="12.7" y="63.5"/>
+<instance part="R5" gate="G$1" x="30.48" y="22.86" rot="R180"/>
 </instances>
 <busses>
@@
 <pinref part="R6" gate="G$1" pin="2"/>
 <pinref part="P+7" gate="1" pin="+12V"/>
-<wire x1="-27.94" y1="73.66" x2="-27.94" y2="66.04" width="0.1524" layer="91"/>
+<wire x1="12.7" y1="60.96" x2="12.7" y2="58.42" width="0.1524" layer="91"/>
 </segment>
 </net>
@@
 <pinref part="SUPPLY3" gate="GND" pin="GND"/>
 </segment>
-<segment>
-<pinref part="R7" gate="G$1" pin="2"/>
-<pinref part="SUPPLY8" gate="GND" pin="GND"/>
-<wire x1="-40.64" y1="45.72" x2="-38.1" y2="45.72" width="0.1524" layer="91"/>
-</segment>
 </net>
 <net name="N" class="0">
@@
 <wire x1="15.24" y1="43.18" x2="15.24" y2="22.86" width="0.1524" layer="91"/>
 <wire x1="25.4" y1="22.86" x2="15.24" y2="22.86" width="0.1524" layer="91"/>
-<pinref part="R5" gate="G$1" pin="E"/>
+<pinref part="R5" gate="G$1" pin="2"/>
 </segment>
 </net>
@@
 <pinref part="Q1" gate="A" pin="E"/>
 <pinref part="T1" gate="A" pin="E"/>
-<wire x1="40.64" y1="22.86" x2="43.18" y2="22.86" width="0.1524" layer="91"/>
-<wire x1="43.18" y1="22.86" x2="68.58" y2="22.86" width="0.1524" layer="91"/>
+<wire x1="35.56" y1="22.86" x2="68.58" y2="22.86" width="0.1524" layer="91"/>
 <wire x1="68.58" y1="22.86" x2="68.58" y2="45.72" width="0.1524" layer="91"/>
 <wire x1="60.96" y1="45.72" x2="68.58" y2="45.72" width="0.1524" layer="91"/>
 <pinref part="J4" gate="-1" pin="1"/>
 <junction x="68.58" y="45.72"/>
-<pinref part="R5" gate="G$1" pin="A"/>
-<pinref part="R5" gate="G$1" pin="S"/>
-<wire x1="33.02" y1="27.94" x2="43.18" y2="27.94" width="0.1524" layer="91"/>
-<wire x1="43.18" y1="27.94" x2="43.18" y2="22.86" width="0.1524" layer="91"/>
+<pinref part="R5" gate="G$1" pin="1"/>
 </segment>
 </net>
@@
 </segment>
 </net>
-<net name="N$4" class="0">
-<segment>
-<pinref part="R1" gate="G$1" pin="1"/>
-<wire x1="5.08" y1="43.18" x2="-12.7" y2="43.18" width="0.1524" layer="91"/>
-<pinref part="IC1" gate="B" pin="OUT"/>
-<wire x1="-12.7" y1="43.18" x2="-12.7" y2="30.48" width="0.1524" layer="91"/>
-<pinref part="R9" gate="G$1" pin="1"/>
-<wire x1="-12.7" y1="30.48" x2="-15.24" y2="30.48" width="0.1524" layer="91"/>
-</segment>
-</net>
 <net name="N$9" class="0">
 <segment>
 <pinref part="IC1" gate="A" pin="+IN"/>
 <pinref part="R2" gate="G$1" pin="2"/>
-<wire x1="15.24" y1="48.26" x2="10.16" y2="48.26" width="0.1524" layer="91"/>
-</segment>
-</net>
-<net name="N$10" class="0">
-<segment>
-<pinref part="IC1" gate="B" pin="+IN"/>
+<wire x1="15.24" y1="48.26" x2="12.7" y2="48.26" width="0.1524" layer="91"/>
 <pinref part="R6" gate="G$1" pin="1"/>
-<pinref part="R7" gate="G$1" pin="1"/>
-<pinref part="R7" gate="G$1" pin="1"/>
-<wire x1="-27.94" y1="55.88" x2="-27.94" y2="45.72" width="0.1524" layer="91"/>
-<junction x="-27.94" y="45.72"/>
-</segment>
-</net>
-<net name="N$11" class="0">
-<segment>
-<pinref part="IC1" gate="B" pin="-IN"/>
-<pinref part="R8" gate="G$1" pin="1"/>
-<pinref part="R9" gate="G$1" pin="2"/>
-<wire x1="-25.4" y1="30.48" x2="-27.94" y2="30.48" width="0.1524" layer="91"/>
-<wire x1="-27.94" y1="30.48" x2="-27.94" y2="40.64" width="0.1524" layer="91"/>
-<junction x="-27.94" y="30.48"/>
+<wire x1="12.7" y1="48.26" x2="10.16" y2="48.26" width="0.1524" layer="91"/>
+<junction x="12.7" y="48.26"/>
 </segment>
 </net>
@@
 <segment>
 <pinref part="IC2" gate="G$1" pin="OUT"/>
-<wire x1="-63.5" y1="43.18" x2="-38.1" y2="43.18" width="0.1524" layer="91"/>
-<pinref part="R8" gate="G$1" pin="2"/>
-<wire x1="-38.1" y1="43.18" x2="-38.1" y2="30.48" width="0.1524" layer="91"/>
-</segment>
-</net>
+<pinref part="R1" gate="G$1" pin="1"/>
+<wire x1="-63.5" y1="43.18" x2="5.08" y2="43.18" width="0.1524" layer="91"/>
+</segment>
+</net>
