File: eagle/ignition4.brd (EAGLE design)
At the start: 152.4 x 152.4 mm, 24 parts, among them IC1 LM358N, IC3 4047N, J1 PIN2F061.100, J2 PIN2F061.100, J3 PIN2F061.100, J4 PIN2F061.100, Q1 MJ2955, T1 2N3055

Commit message: fix some things on dbd board
Parts:
- C7: value 1000pF -> 500pF
- IC1: value LM358N -> LT1352PA; device linear:DIL08 -> linear-technology:DIL08
- R2: value 10k -> 0
- R6: value 10k -> 30k
- R8: value 30k -> 10k
- moved C4 3.25 mm to (55.1, 22.9)
- moved IC1 0.25 mm to (32.3, 102.4)
Routing:
- net +12V: track 173.9 -> 245.1 mm, vias 0 -> 1
