File: eagle/ignition4.sch (EAGLE design)
At the start: 24 parts, among them IC1 LM358N, IC3 4047N, J1 PIN2F061.100, J2 PIN2F061.100, J3 PIN2F061.100, J4 PIN2F061.100, Q1 MJ2955, T1 2N3055

Commit message: fix some things on dbd board
Parts:
- C7: value 1000pF -> 500pF
- IC1: value LM358N -> LT1352PA; device linear:LM358N -> linear-technology:LT1352PA
- R2: value 10k -> 0
- R6: value 10k -> 30k
- R8: value 30k -> 10k
Connections:
- net +12V: now also IC1A.V+; no longer IC1P.V+
- net -12V: now also IC1A.V-; no longer IC1P.V-
Other:
- moved on the sheet: IC1B
Changed lines of the file:
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@@
 </classes>
 <parts>
-<part name="IC1" library="linear" deviceset="LM358" device="N"/>
 <part name="T1" library="transistor" deviceset="2N3055" device=""/>
 <part name="Q1" library="transistor-pnp" deviceset="MJ2955" device=""/>
@@
 <part name="C5" library="rcl" deviceset="C-US" device="050-035X075"/>
 <part name="C6" library="rcl" deviceset="CPOL-US" device="E5-5"/>
-<part name="R2" library="resistor" deviceset="R-US_" device="0207/15" value="10k"/>
+<part name="R2" library="resistor" deviceset="R-US_" device="0207/15" value="0"/>
 <part name="SUPPLY3" library="supply2" deviceset="GND" device=""/>
-<part name="R6" library="resistor" deviceset="R-US_" device="0207/12" value="10k"/>
+<part name="R6" library="resistor" deviceset="R-US_" device="0207/12" value="30k"/>
 <part name="R7" library="resistor" deviceset="R-US_" device="0207/10" value="10k"/>
-<part name="R8" library="resistor" deviceset="R-US_" device="0207/10" value="30k"/>
+<part name="R8" library="resistor" deviceset="R-US_" device="0207/10" value="10k"/>
 <part name="R9" library="resistor" deviceset="R-US_" device="0207/10" value="10k"/>
 <part name="P+7" library="supply1" deviceset="+12V" device=""/>
 <part name="SUPPLY8" library="supply2" deviceset="GND" device=""/>
 <part name="IC3" library="40xx" deviceset="4047" device="N"/>
-<part name="C7" library="rcl" deviceset="C-US" device="075-042X103" value="1000pF"/>
+<part name="C7" library="rcl" deviceset="C-US" device="075-042X103" value="500pF"/>
 <part name="SUPPLY9" library="supply2" deviceset="GND" device=""/>
 <part name="P+8" library="supply1" deviceset="+12V" device=""/>
@@
 <part name="R3" library="piher" deviceset="PC16S" device="" value="20K"/>
 <part name="R4" library="piher" deviceset="PC16S" device="" value="250K"/>
+<part name="IC1" library="linear-technology" deviceset="LT1352" device="PA"/>
 </parts>
 <sheets>
@@
 </plain>
 <instances>
-<instance part="IC1" gate="A" x="22.86" y="45.72"/>
 <instance part="T1" gate="A" x="58.42" y="50.8"/>
 <instance part="Q1" gate="A" x="58.42" y="40.64"/>
@@
 <instance part="J1" gate="-1" x="106.68" y="172.72"/>
 <instance part="J2" gate="-1" x="106.68" y="152.4"/>
-<instance part="IC1" gate="P" x="22.86" y="45.72"/>
 <instance part="P+2" gate="1" x="22.86" y="55.88"/>
 <instance part="P-2" gate="1" x="22.86" y="35.56"/>
@@
 <instance part="C6" gate="G$1" x="-5.08" y="127"/>
 <instance part="R2" gate="G$1" x="5.08" y="48.26"/>
-<instance part="IC1" gate="B" x="-20.32" y="43.18"/>
 <instance part="SUPPLY3" gate="GND" x="-5.08" y="48.26" rot="R270"/>
 <instance part="R6" gate="G$1" x="-27.94" y="60.96" rot="R90"/>
@@
 <instance part="R3" gate="G$1" x="25.4" y="27.94"/>
 <instance part="R4" gate="G$1" x="-104.14" y="12.7"/>
+<instance part="IC1" gate="A" x="25.4" y="45.72"/>
+<instance part="IC1" gate="B" x="-17.78" y="43.18"/>
 </instances>
 <busses>
@@
 </segment>
 <segment>
-<pinref part="IC1" gate="P" pin="V+"/>
-<pinref part="P+2" gate="1" pin="+12V"/>
-</segment>
-<segment>
 <pinref part="T1" gate="A" pin="C"/>
 <pinref part="P+3" gate="1" pin="+12V"/>
@@
 <pinref part="P+11" gate="1" pin="+12V"/>
 <wire x1="-78.74" y1="25.4" x2="-73.66" y2="25.4" width="0.1524" layer="91"/>
+</segment>
+<segment>
+<pinref part="P+2" gate="1" pin="+12V"/>
+<pinref part="IC1" gate="A" pin="V+"/>
 </segment>
 </net>
@@
 </segment>
 <segment>
-<pinref part="IC1" gate="P" pin="V-"/>
-<pinref part="P-2" gate="1" pin="-12V"/>
-</segment>
-<segment>
 <pinref part="Q1" gate="A" pin="C"/>
 <pinref part="P-3" gate="1" pin="-12V"/>
 <wire x1="60.96" y1="30.48" x2="60.96" y2="35.56" width="0.1524" layer="91"/>
+</segment>
+<segment>
+<pinref part="P-2" gate="1" pin="-12V"/>
+<pinref part="IC1" gate="A" pin="V-"/>
 </segment>
 </net>
@@
 <net name="N$1" class="0">
 <segment>
-<pinref part="IC1" gate="A" pin="-IN"/>
 <pinref part="R1" gate="G$1" pin="2"/>
 <wire x1="15.24" y1="43.18" x2="15.24" y2="22.86" width="0.1524" layer="91"/>
 <wire x1="15.24" y1="22.86" x2="20.32" y2="22.86" width="0.1524" layer="91"/>
 <pinref part="R3" gate="G$1" pin="1A"/>
+<pinref part="IC1" gate="A" pin="-IN"/>
+<junction x="15.24" y="43.18"/>
 </segment>
 </net>
@@
 <wire x1="38.1" y1="50.8" x2="38.1" y2="45.72" width="0.1524" layer="91"/>
 <wire x1="38.1" y1="40.64" x2="38.1" y2="45.72" width="0.1524" layer="91"/>
+<wire x1="38.1" y1="45.72" x2="35.56" y2="45.72" width="0.1524" layer="91"/>
 <pinref part="IC1" gate="A" pin="OUT"/>
-<wire x1="38.1" y1="45.72" x2="30.48" y2="45.72" width="0.1524" layer="91"/>
+<wire x1="35.56" y1="45.72" x2="30.48" y2="45.72" width="0.1524" layer="91"/>
+<junction x="35.56" y="45.72"/>
 </segment>
 </net>
@@
 <segment>
 <pinref part="R1" gate="G$1" pin="1"/>
-<wire x1="5.08" y1="43.18" x2="-12.7" y2="43.18" width="0.1524" layer="91"/>
-<pinref part="IC1" gate="B" pin="OUT"/>
+<wire x1="5.08" y1="43.18" x2="-7.62" y2="43.18" width="0.1524" layer="91"/>
+<wire x1="-7.62" y1="43.18" x2="-12.7" y2="43.18" width="0.1524" layer="91"/>
 <wire x1="-12.7" y1="43.18" x2="-12.7" y2="30.48" width="0.1524" layer="91"/>
 <pinref part="R9" gate="G$1" pin="1"/>
 <wire x1="-12.7" y1="30.48" x2="-15.24" y2="30.48" width="0.1524" layer="91"/>
+<pinref part="IC1" gate="B" pin="OUT"/>
+<junction x="-7.62" y="43.18"/>
 </segment>
 </net>
 <net name="N$9" class="0">
 <segment>
-<pinref part="IC1" gate="A" pin="+IN"/>
 <pinref part="R2" gate="G$1" pin="2"/>
 <wire x1="15.24" y1="48.26" x2="10.16" y2="48.26" width="0.1524" layer="91"/>
+<pinref part="IC1" gate="A" pin="+IN"/>
 </segment>
 </net>
 <net name="N$10" class="0">
 <segment>
-<pinref part="IC1" gate="B" pin="+IN"/>
 <pinref part="R6" gate="G$1" pin="1"/>
 <pinref part="R7" gate="G$1" pin="1"/>
@@
 <wire x1="-27.94" y1="55.88" x2="-27.94" y2="45.72" width="0.1524" layer="91"/>
 <junction x="-27.94" y="45.72"/>
+<pinref part="IC1" gate="B" pin="+IN"/>
 </segment>
 </net>
 <net name="N$11" class="0">
 <segment>
-<pinref part="IC1" gate="B" pin="-IN"/>
 <pinref part="R8" gate="G$1" pin="1"/>
 <pinref part="R9" gate="G$1" pin="2"/>
@@
 <wire x1="-27.94" y1="30.48" x2="-27.94" y2="40.64" width="0.1524" layer="91"/>
 <junction x="-27.94" y="30.48"/>
-</segment>
-</net>
+<pinref part="IC1" gate="B" pin="-IN"/>
+</segment>
+</net>
